File: GP1247AI.kicad_sch (KiCad schematic)
At the start: 15 parts, among them J1 Conn_02x05_Odd_Even, J2 Conn_02x05_Odd_Even, U2 B0505S-2WR3

Commit message: Added onboard MCU
Parts:
- removed D1: 3v3, Diode_SMD:D_SOD-123, symbol Device:D_Zener
- removed J2: Conn_02x05_Odd_Even, Connector_PinHeader_2.54mm:PinHeader_2x05_P2.54mm_Vertical, symbol Connector_Generic:Conn_02x05_Odd_Even
- added BT1: Battery_Cell, CustomFootprints:QIJEY CR2032-BS-6-1, symbol Device:Battery_Cell
- added C10, C11, C7, C8, C9: 100n, Capacitor_SMD:C_0603_1608Metric, symbol Device:C_Small
- added C12, C18, C19, C25, C26, C27, C28, C6: 22u, Capacitor_SMD:C_0603_1608Metric, symbol Device:C
- added C13: 10n, Capacitor_SMD:C_0603_1608Metric, symbol Device:C
- added C14: 2u2, Capacitor_SMD:C_0603_1608Metric, symbol Device:C
- added C15, C24: 100n, Capacitor_SMD:C_0603_1608Metric, symbol Device:C
- added C16, C17: 20p, Capacitor_SMD:C_0603_1608Metric, symbol Device:C_Small
- added C20, C21: 5p, Capacitor_SMD:C_0603_1608Metric, symbol Device:C_Small
- added C22, C23: 2u2, Capacitor_SMD:C_0603_1608Metric, symbol Device:C_Small
- added J2: Conn_01x04_Pin, Connector_PinHeader_2.54mm:PinHeader_1x04_P2.54mm_Vertical, symbol Connector:Conn_01x04_Pin
- added J3: USB_C_Receptacle_USB2.0_14P, CustomFootprints:USB_TYPE-C-31-M-12, symbol Connector:USB_C_Receptacle_USB2.0_14P
- added J4: Conn_01x04_Socket, Connector_PinSocket_2.54mm:PinSocket_1x04_P2.54mm_Horizontal, symbol Connector:Conn_01x04_Socket
- added JP1: Jumper_2_Small_Bridged, Connector_PinHeader_2.54mm:PinHeader_1x02_P2.54mm_Vertical, symbol Jumper:Jumper_2_Small_Bridged
- added N1: Housing_Pad, TestPoint:TestPoint_Pad_2.0x2.0mm, symbol Mechanical:Housing_Pad
- added R10, R4, R5, R9: 5k1, Resistor_SMD:R_0603_1608Metric, symbol Device:R
- added R2, R3, R6, R7, R8: 1k, Resistor_SMD:R_0603_1608Metric, symbol Device:R
- added SW1: SW_Push, CustomFootprints:Korean Hroparts Elec K2-1107ST-A4DW-06, symbol Switch:SW_Push
- added SW2: SW-520D, CustomFootprints:SW-520D, symbol Switch:SW_SPST
- added TP1, TP2: TestPoint, TestPoint:TestPoint_Pad_D1.5mm, symbol Connector:TestPoint
- added TP3, TP4, TP5, TP6, TP7: TestPoint, CustomFootprints:TestPoint_Keystone_5019_Miniature, symbol Connector:TestPoint
- added U3: STM32F405RGTx, Package_QFP:LQFP-64_10x10mm_P0.5mm, symbol MCU_ST_STM32F4:STM32F405RGTx
- added U4: TLV75733PDBV, Package_TO_SOT_SMD:SOT-23-5, symbol Regulator_Linear:TLV75733PDBV
- added U5: USBLC6-2SC6, Package_TO_SOT_SMD:SOT-23-6, symbol Power_Protection:USBLC6-2SC6
- added U6: W25Q128JVSIQ, Package_SO:SOIC-8_5.3x5.3mm_P1.27mm, symbol Memory_Flash:W25Q128JVS
- added Y1: 8 MHz, Crystal:Crystal_SMD_5032-2Pin_5.0x3.2mm, symbol Device:Crystal
- added Y2: 32.768 kHz, CustomFootprints:SMD3215-2P, symbol Device:Crystal
- J1: footprint Connector_PinHeader_2.54mm:PinHeader_2x05_P2.54mm_Vertical -> Connector_IDC:IDC-Header_2x05_P2.54mm_Vertical; LCSC PART # C42431818 -> (none)
- R1: value 10k -> 5k1; LCSC PART # C49652949 -> C23186
Connections:
- net +3V3: now also J1.2 (Pin_2), C10.1, C11.1, C12.1, C13.1, C14.1, C19.1, C24.1, C8.1, C9.1, J2.1 (Pin_1), JP1.1 (A), R10.1, R2.1, R9.1, U3.13 (VDDA), U3.19 (VDD), U3.32 (VDD), U3.48 (VDD), U3.64 (VDD), U4.5 (OUT), U6.8 (VCC); no longer J1.1 (Pin_1)
- net +5V: now also J1.1 (Pin_1), C18.1, J3.A4 (VBUS), J3.A9 (VBUS), J3.B4 (VBUS), J3.B9 (VBUS), U4.1 (IN), U4.3 (EN), U5.5 (VBUS); no longer J1.7 (Pin_7)
- net F-: now also JP1.2 (B)
- net GND: now also J1.7 (Pin_7), BT1.2 (-), C10.2, C11.2, C12.2, C13.2, C14.2, C15.1, C16.2, C17.2, C18.2, C19.2, C20.2, C21.2, C22.2, C23.2, C24.2, C25.2, C26.2, C27.2, C28.2, C6.2, C7.2, C8.2, C9.2, J2.4 (Pin_4), J3.A1 (GND), J3.A12 (GND), J3.B1 (GND), J3.B12 (GND), J4.1 (Pin_1), R4.2, R5.2, SW1.1, SW2.1 (A), TP7.1, U3.12 (VSSA), U3.18 (VSS), U3.63 (VSS), U4.2 (GND), U5.2 (GND), U6.4 (GND)
- net CLK renamed DISP_CLK
- net DISP_CLK: now also U3.29 (PB10)
- net CS renamed DISP_CS
- net DISP_CS: now also U3.33 (PB12)
- net DIO renamed DISP_DIO
- net DISP_DIO: now also U3.36 (PB15)
- net RST: no longer names the net of U1.10 (~{RESET})
- net RST: now also R2.2; no longer J1.2 (Pin_2)
- new net: J4.2 (Pin_2), R8.1
- new net: J4.3 (Pin_3), R7.1
- new net: J4.4 (Pin_4), R6.1
- new net: R3.1, SW2.2 (B)
- new net: C15.2, SW1.2, U3.7 (NRST)
- new net: J3.S1 (SHIELD), N1.1 (PAD)
- new net B0: TP1.1, U3.60 (BOOT0)
- new net CC1: J3.A5 (CC1), R4.1
- new net CC2: J3.B5 (CC2), R5.1
- new net CD+: J3.A6 (D+), J3.B6 (D+), U5.3 (I/O2)
- new net CD-: J3.A7 (D-), J3.B7 (D-), U5.1 (I/O1)
- new net D+: U3.45 (PA12), U5.4 (I/O2)
- new net D-: U3.44 (PA11), U5.6 (I/O1)
- new net FLASH_CLK: TP4.1, U3.51 (PC10), U6.6 (CLK)
- new net FLASH_CS: TP3.1, U3.50 (PA15), U6.1 (~{CS})
- new net FLASH_MISO: TP6.1, U3.52 (PC11), U6.2 (DO/IO_{1})
- new net FLASH_MOSI: TP5.1, U3.53 (PC12), U6.5 (DI/IO_{0})
- new net HOLD: R10.2, U6.7 (~{HOLD}/~{RESET}/IO_{3})
- new net MCO: TP2.1, U3.41 (PA8)
- new net OSC32_IN: C20.1, U3.3 (PC14), Y2.1
- new net OSC32_OUT: C21.1, U3.4 (PC15), Y2.2
- new net OSC_IN: C16.1, U3.5 (PH0), Y1.2
- new net OSC_OUT: C17.1, U3.6 (PH1), Y1.1
- new net SW1: C26.1, R6.2, U3.25 (PC5)
- new net SW2: C27.1, R7.2, U3.24 (PC4)
- new net SW3: C28.1, R8.2, U3.23 (PA7)
- new net SWCLK: J2.3 (Pin_3), U3.49 (PA14)
- new net SWDIO: J2.2 (Pin_2), U3.46 (PA13)
- new net TILT: C25.1, R3.2, U3.26 (PB0)
- new net VBAT: BT1.1 (+), C6.1, C7.1, U3.1 (VBAT)
- new net VCAP_1: C22.1, U3.31 (VCAP_1)
- new net VCAP_2: C23.1, U3.47 (VCAP_2)
- new net WP: R9.2, U6.3 (~{WP}/IO_{2})
- no-connect marks 1 -> 32
Other:
- note added: "16MiB Flash"
- note added: "256 byte page (x16 per sector) 4 KiB sector (x16 per block) 64 KiB block (x256)"
- note added: "Analog Decoupling"
- note added: "Connector"
- note added: "Cs = 10pF (stray) C = 2 * (Cl - Cs) Where Cl = Cl1 = Cl2 C = 2 * (20 - 10) = 20 pF (8MHz) C = 2 * (12.5 - 10) = 5 pF (32kHz)"
- note added: "For debugging SPI timing"
- note added: "STM32F405"
- note added: "Switches"
- note added: "Test Points"
- note added: "Tilt switch is closed when the PCB is right side up"
- note added: "To support an external MCU if the on-board MCU is not populated"
- note added: "USB-C"
- note removed: "Connectors"
- note removed: "Pair With C843271"
- moved on the sheet: C1, C2, C3, C4, C5, H1, H2, H3, H4, J1, U1, U2
