File: boost1.kicad_sch (KiCad schematic)
At the start: 18 parts, among them Q1 G1003B-23, U3 LM3478MA

Commit message: Added onboard MCU
Parts:
- removed C6: 22u, Capacitor_THT:CP_Radial_D6.3mm_P2.50mm, symbol Device:C_Polarized
- removed JP1: Jumper_2_Small_Bridged, Connector_PinHeader_2.54mm:PinHeader_1x02_P2.54mm_Vertical, symbol Jumper:Jumper_2_Small_Bridged
- removed R8: 1k, Resistor_SMD:R_0603_1608Metric, symbol Device:R
- added C29: 22u, Capacitor_SMD:C_0603_1608Metric, symbol Device:C
- added JP2: Jumper_2_Small_Bridged, Connector_PinHeader_2.54mm:PinHeader_1x02_P2.54mm_Vertical, symbol Jumper:Jumper_2_Small_Bridged
- added R17: 1k, Resistor_SMD:R_0603_1608Metric, symbol Device:R
- renumbered C7 to C30, C8 to C31, C9 to C32, C10 to C33, D2 to D1, R2 to R11, R3 to R12, R4 to R13, R5 to R14, R6 to R15, R7 to R16, U3 to U7
Connections:
- net +50V: now also JP2.2 (B)
- net +5V: now also C29.1
- net 50V_BOOST: now also JP2.1 (A)
- net GND: now also C29.2, R17.2
- net at C32.2: now also R17.1
Other:
- note added: "Dissipation factor is usually 10% on 0603 ceramics This will correlate to ~1.6mohm ESR at 460kHZ So the cap can easily handle the RMS current without heating"
