File: PCB/GP1247AI.kicad_sch (KiCad schematic)
At the start: 68 parts, among them J1 Conn_02x05_Odd_Even, J2 Conn_01x04_Pin, J3 USB_C_Receptacle_USB2.0_14P, J4 Conn_01x04_Socket, SW1 SW_Push, SW2 SW-520D, U2 B0505S-2WR3, U3 STM32F405RGTx, U4 TLV75733PDBV, U5 USBLC6-2SC6, U6 W25Q128JVSIQ, Y1 8 MHz, Y2 32.768 kHz

Commit message: Fixed floating boot0
Parts:
- removed TP1: TestPoint, TestPoint:TestPoint_Pad_D1.5mm, symbol Connector:TestPoint
- added R12: 5k1, Resistor_SMD:R_0603_1608Metric, symbol Device:R
- U2: renamed from U1; value ~ -> (none)
- renumbered C28 to C10, C19 to C11, C20 to C12, C15 to C13, C16 to C14, C21 to C15, C17 to C16, C22 to C17, C23 to C18, C6 to C19, C7 to C20, C8 to C21, C9 to C22, C10 to C23, C11 to C24, C12 to C25, C24 to C26, C13 to C27, C14 to C28, C25 to C3, C3 to C4, C26 to C5, C18 to C6, C4 to C7, C27 to C8, C5 to C9, H3 to H2, H2 to H3, J3 to J1, J1 to J2, J4 to J3, J2 to J4, R4 to R1, R7 to R10, R8 to R11, R10 to R13, R11 to R14, R5 to R2, R2 to R3, R9 to R4, R12 to R5, R13 to R6, R1 to R7, R3 to R8, R6 to R9, SW2 to SW1, SW1 to SW2, TP2 to TP1, TP3 to TP2, TP4 to TP3, TP5 to TP4, TP6 to TP5, TP7 to TP6, U5 to U1, U4 to U3, U2 to U4, U3 to U5, Y2 to Y1, Y1 to Y2
Connections:
- net GND: now also R12.1
- net B0 renamed BT0
- net BT0: now also R12.2
