File: PCB/boost1.kicad_sch (KiCad schematic)
At the start: 18 parts, among them Q1 G1003B-23, U7 LM3478MA

Commit message: Fixed floating boot0
Parts:
- renumbered C30 to C29, C32 to C30, C29 to C31, C33 to C32, C31 to C33, R14 to R15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
